File: 4dof-arm/4dof-arm.kicad_pcb (KiCad board)
At the start: 2 copper layers, 73 x 61.7 mm, 20 parts, among them J1 Servo-0, J2 Servo-1, J3 Servo-2, J4 Servo-3, J5 I2C, J6 I2C, J7 UART, J8 Reset, U1 bluepill-stm32f103c8, U2 NRF24L01_Breakout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

Commit message: 4dof-arm: Fix nRF24L01+ CE and IRQ signal
Connections:
- U1 pad 23: /nRF_CE -> unconnected-(U1-PC14-Pad23)
- U1 pad 24: /nRF_IRQ -> unconnected-(U1-PC15-Pad24)
- U1 pad 27: unconnected-(U1-PA2_TXD1-Pad27) -> /nRF_CE
- U1 pad 28: unconnected-(U1-PA3_RXD1-Pad28) -> /nRF_IRQ
Routing:
- net /nRF_IRQ: track 64.6 -> 45.6 mm, vias 1 -> 0
- net /nRF_CE: track 52.8 -> 41.9 mm
Changed lines of the file:
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@@
   (net 25 "unconnected-(U1-PA0_A0-Pad25)")
   (net 26 "unconnected-(U1-PA1_A1-Pad26)")
-  (net 27 "unconnected-(U1-PA2_TXD1-Pad27)")
-  (net 28 "unconnected-(U1-PA3_RXD1-Pad28)")
+  (net 27 "unconnected-(U1-PC14-Pad23)")
+  (net 28 "unconnected-(U1-PC15-Pad24)")
   (net 29 "unconnected-(U1-PA4_A2_CS1-Pad29)")
   (net 30 "unconnected-(U1-PA5_A3_SCLK1-Pad30)")
@@
       (net 24 "unconnected-(U1-PC13_LED0-Pad22)") (pinfunction "PC13_LED0") (pintype "unspecified"))
     (pad "23" thru_hole circle (at -15.24 -43.18 90) (size 1.6 1.6) (drill 0.8) (layers "*.Cu" "*.Mask")
-      (net 37 "/nRF_CE") (pinfunction "PC14") (pintype "unspecified"))
+      (net 27 "unconnected-(U1-PC14-Pad23)") (pinfunction "PC14") (pintype "unspecified"))
     (pad "24" thru_hole circle (at -15.24 -40.64 90) (size 1.6 1.6) (drill 0.8) (layers "*.Cu" "*.Mask")
-      (net 38 "/nRF_IRQ") (pinfunction "PC15") (pintype "unspecified"))
+      (net 28 "unconnected-(U1-PC15-Pad24)") (pinfunction "PC15") (pintype "unspecified"))
     (pad "25" thru_hole circle (at -15.24 -38.1 90) (size 1.6 1.6) (drill 0.8) (layers "*.Cu" "*.Mask")
       (net 25 "unconnected-(U1-PA0_A0-Pad25)") (pinfunction "PA0_A0") (pintype "unspecified"))
@@
       (net 26 "unconnected-(U1-PA1_A1-Pad26)") (pinfunction "PA1_A1") (pintype "unspecified"))
     (pad "27" thru_hole circle (at -15.24 -33.02 90) (size 1.6 1.6) (drill 0.8) (layers "*.Cu" "*.Mask")
-      (net 27 "unconnected-(U1-PA2_TXD1-Pad27)") (pinfunction "PA2_TXD1") (pintype "unspecified"))
+      (net 37 "/nRF_CE") (pinfunction "PA2_TXD1") (pintype "unspecified"))
     (pad "28" thru_hole circle (at -15.24 -30.48 90) (size 1.6 1.6) (drill 0.8) (layers "*.Cu" "*.Mask")
-      (net 28 "unconnected-(U1-PA3_RXD1-Pad28)") (pinfunction "PA3_RXD1") (pintype "unspecified"))
+      (net 38 "/nRF_IRQ") (pinfunction "PA3_RXD1") (pintype "unspecified"))
     (pad "29" thru_hole circle (at -15.24 -27.94 90) (size 1.6 1.6) (drill 0.8) (layers "*.Cu" "*.Mask")
       (net 29 "unconnected-(U1-PA4_A2_CS1-Pad29)") (pinfunction "PA4_A2_CS1") (pintype "unspecified"))
@@
   (segment (start 86.195 40.8678) (end 88.5072 43.18) (width 0.25) (layer "F.Cu") (net 36))
   (segment (start 95.25 43.18) (end 97.1675 45.0975) (width 0.25) (layer "F.Cu") (net 36))
-  (segment (start 38.735 65.405) (end 35.56 62.23) (width 0.25) (layer "F.Cu") (net 37))
   (segment (start 71.12 76.2) (end 60.325 65.405) (width 0.25) (layer "F.Cu") (net 37))
-  (segment (start 35.56 62.23) (end 35.56 60.96) (width 0.25) (layer "F.Cu") (net 37))
-  (segment (start 60.325 65.405) (end 38.735 65.405) (width 0.25) (layer "F.Cu") (net 37))
+  (segment (start 50.165 65.405) (end 45.72 60.96) (width 0.25) (layer "F.Cu") (net 37))
+  (segment (start 60.325 65.405) (end 50.165 65.405) (width 0.25) (layer "F.Cu") (net 37))
   (via (at 71.12 76.2) (size 0.8) (drill 0.4) (layers "F.Cu" "B.Cu") (net 37))
   (segment (start 81.28 76.2) (end 71.12 76.2) (width 0.25) (layer "B.Cu") (net 37))
-  (segment (start 81.915 83.185) (end 45.085 83.185) (width 0.25) (layer "F.Cu") (net 38))
-  (segment (start 83.82 81.28) (end 81.915 83.185) (width 0.25) (layer "F.Cu") (net 38))
-  (segment (start 39.37 70.485) (end 38.1 69.215) (width 0.25) (layer "F.Cu") (net 38))
-  (segment (start 39.37 77.47) (end 39.37 70.485) (width 0.25) (layer "F.Cu") (net 38))
-  (segment (start 45.085 83.185) (end 39.37 77.47) (width 0.25) (layer "F.Cu") (net 38))
-  (via (at 38.1 69.215) (size 0.8) (drill 0.4) (layers "F.Cu" "B.Cu") (net 38))
-  (segment (start 38.1 69.215) (end 38.1 60.96) (width 0.25) (layer "B.Cu") (net 38))
+  (segment (start 80.645 83.185) (end 81.915 83.185) (width 0.25) (layer "F.Cu") (net 38))
+  (segment (start 52.255 64.955) (end 62.415 64.955) (width 0.25) (layer "F.Cu") (net 38))
+  (segment (start 62.415 64.955) (end 80.645 83.185) (width 0.25) (layer "F.Cu") (net 38))
+  (segment (start 81.915 83.185) (end 83.82 81.28) (width 0.25) (layer "F.Cu") (net 38))
+  (segment (start 48.26 60.96) (end 52.255 64.955) (width 0.25) (layer "F.Cu") (net 38))
   (segment (start 98.425 39.37) (end 99.06 40.005) (width 0.25) (layer "F.Cu") (net 39))
   (segment (start 98.4239 60.9589) (end 97.1675 60.9589) (width 0.25) (layer "F.Cu") (net 39))
